File: pcbs/backplane/cptrep_8500_backplane/cptrep_8500_backplane/cptrep_8500_backplane.kicad_sch (KiCad schematic)
At the start: 5 parts, among them J1 Conn_02x50_Row_Letter_First, J2 Conn_02x50_Row_Letter_First, J3 Conn_02x50_Row_Letter_First, J4 Conn_02x50_Row_Letter_First, J5 Conn_02x50_Row_Letter_First

Commit message: "Update"
Parts:
- removed J1, J2, J3, J4, J5: Conn_02x50_Row_Letter_First, Connector_Samtec_HLE_THT:Samtec_HLE-150-02-xx-DV-TE_2x50_P2.54mm_Horizontal, symbol Connector_Generic:Conn_02x50_Row_Letter_First
- added D1, D2, D3, D4, D5: LED, symbol Device:LED
- added R1: 4k7, symbol Device:R_Small
- added R2, R4: 2k2, symbol Device:R_Small
- added R3, R5: 1k, symbol Device:R_Small
Connections:
- new net: D3.2 (A), R4.2
- new net: D5.2 (A), R5.2
- new net: D1.2 (A), R1.2
- new net: D2.2 (A), R2.2
- new net: D4.2 (A), R3.2
- new net +12V: R2.1
- new net +24V: R1.1
- new net +5V: R3.1
- new net -12V: D3.1 (K)
- new net -5V: D5.1 (K)
- new net GND: D1.1 (K), D2.1 (K), D4.1 (K), R4.1, R5.1
Other:
- added sheet BPCONN1 (bpconn1.kicad_sch)
- added sheet BPCONN2 (bpconn2.kicad_sch)
- added sheet BPCONN3 (bpconn3.kicad_sch)
- added sheet BPCONN4 (bpconn4.kicad_sch)
- added sheet BPCONN5 (bpconn5.kicad_sch)

Commit message: "Update"
Parts:
- added C1, C2: C_Small, Capacitor_SMD:C_0805_2012Metric_Pad1.18x1.45mm_HandSolder, symbol Device:C_Small
- added J10, J7, J8, J9: Screw_Terminal_01x04, TerminalBlock_Phoenix:TerminalBlock_Phoenix_MKDS-1,5-4_1x04_P5.00mm_Horizontal, symbol Connector:Screw_Terminal_01x04
- added SW1: SW_Push, Button_Switch_THT:SW_PUSH_6mm, symbol Switch:SW_Push
- added U1: LM7905_TO220, Package_TO_SOT_THT:TO-220-3_Horizontal_TabDown, symbol Regulator_Linear:LM7905_TO220
- D1, D2, D3, D4, D5: footprint (none) -> LED_SMD:LED_0805_2012Metric_Pad1.15x1.40mm_HandSolder
- R1, R2, R3, R4, R5: footprint (none) -> Resistor_SMD:R_0805_2012Metric_Pad1.20x1.40mm_HandSolder
Connections:
- net +12V: now also J9.1 (Pin_1)
- net +5V: now also J9.4 (Pin_4)
- net -12V: now also C2.1, J8.4 (Pin_4), U1.2 (VI)
- net -5V: now also C1.1, U1.3 (VO)
- net GND: now also C1.2, C2.2, J7.1 (Pin_1), J8.2 (Pin_2), J8.3 (Pin_3), J9.2 (Pin_2), J9.3 (Pin_3), U1.1 (GND)
- new net AUD: J7.3 (Pin_3)
- new net /BP83: J7.4 (Pin_4)
- new net /BP85: J8.1 (Pin_1)
- new net /CLEAR: J7.2 (Pin_2)

Commit message: "Update"
Connections:
- net +24V: now also J10.1 (Pin_1)
- net GND: now also J10.4 (Pin_4)
Changed lines of the file:
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@@
+	(wire
+		(pts
+			(xy 74.93 150.495) (xy 74.93 146.685)
+		)
+		(stroke
+			(width 0)
+			(type default)
+		)
+	)
 	(wire
 		(pts
@@
 	(wire
 		(pts
+			(xy 57.785 150.495) (xy 74.93 150.495)
+		)
+		(stroke
+			(width 0)
+			(type default)
+		)
+	)
+	(wire
+		(pts
+			(xy 57.785 158.115) (xy 62.865 158.115)
+		)
+		(stroke
+			(width 0)
+			(type default)
+		)
+	)
+	(wire
+		(pts
 			(xy 68.58 28.575) (xy 68.58 31.75)
 		)
@@
 		(pts
 			(xy 40.005 20.955) (xy 40.005 23.495)
+		)
+		(stroke
+			(width 0)
+			(type default)
+		)
+	)
+	(wire
+		(pts
+			(xy 62.865 158.115) (xy 62.865 161.925)
 		)
 		(stroke
@@
 	(symbol
 		(lib_id "power:GND")
+		(at 62.865 161.925 0)
+		(mirror y)
+		(unit 1)
+		(exclude_from_sim no)
+		(in_bom yes)
+		(on_board yes)
+		(dnp no)
+		(fields_autoplaced yes)
+		(property "Reference" "#PWR091"
+			(at 62.865 168.275 0)
+			(effects
+				(font
+					(size 1.27 1.27)
+				)
+				(hide yes)
+			)
+		)
+		(property "Value" "GND"
+			(at 62.865 167.005 0)
+			(effects
+				(font
+					(size 1.27 1.27)
+				)
+			)
+		)
+		(property "Footprint" ""
+			(at 62.865 161.925 0)
+			(effects
+				(font
+					(size 1.27 1.27)
+				)
+				(hide yes)
+			)
+		)
+		(property "Datasheet" ""
+			(at 62.865 161.925 0)
+			(effects
+				(font
+					(size 1.27 1.27)
+				)
+				(hide yes)
+			)
+		)
+		(property "Description" "Power symbol creates a global label with name \"GND\" , ground"
+			(at 62.865 161.925 0)
+			(effects
+				(font
+					(size 1.27 1.27)
+				)
+				(hide yes)
+			)
+		)
+		(pin "1"
+		)
+		(instances
+			(project "cptrep_8500_backplane"
+				(path "/6bc3ef00-9758-4385-9185-3572b301e705"
+					(reference "#PWR091")
+					(unit 1)
+				)
+			)
+		)
+	)
+	(symbol
+		(lib_id "power:GND")
 		(at 43.18 87.63 0)
 		(mirror y)
@@
 					(unit 1)
 				)
+			)
+		)
+	)
+	(symbol
+		(lib_id "power:+24V")
+		(at 74.93 146.685 0)
+		(unit 1)
+		(exclude_from_sim no)
+		(in_bom yes)
+		(on_board yes)
+		(dnp no)
+		(fields_autoplaced yes)
+		(property "Reference" "#PWR090"
+			(at 74.93 150.495 0)
+			(effects
+				(font
+					(size 1.27 1.27)
+				)
+				(hide yes)
+			)
+		)
+		(property "Value" "+24V"
+			(at 74.93 142.24 0)
+			(effects
+				(font
+					(size 1.27 1.27)
+				)
+			)
+		)
+		(property "Footprint" ""
+			(at 74.93 146.685 0)
+			(effects
+				(font
+					(size 1.27 1.27)
+				)
+				(hide yes)
+			)
+		)
+		(property "Datasheet" ""
+			(at 74.93 146.685 0)
+			(effects
+				(font
+					(size 1.27 1.27)
+				)
+				(hide yes)
+			)
+		)
+		(property "Description" "Power symbol creates a global label with name \"+24V\""
+			(at 74.93 146.685 0)
+			(effects
+				(font
+					(size 1.27 1.27)
+				)
+				(hide yes)
+			)
+		)
+		(pin "1"
+		)
+		(instances
+			(project "cptrep_8500_backplane"
+				(path "/6bc3ef00-9758-4385-9185-3572b301e705"
+					(reference "#PWR090")
+					(unit 1)
+				)

Commit message: "Update"
Parts:
- added J6: Conn_01x02_Pin, Connector_PinSocket_2.54mm:PinSocket_1x02_P2.54mm_Vertical, symbol Connector:Conn_01x02_Pin
- added R6: 27R, Resistor_SMD:R_0805_2012Metric_Pad1.20x1.40mm_HandSolder, symbol Device:R_Small
Connections:
- net AUD: now also J6.1 (Pin_1)
- net GND: now also J6.2 (Pin_2), R6.1
- net /CLEAR: now also SW1.2
- net at SW1.1: now also R6.2
Other:
- note added: "Audio output"
- note added: "RESET"
- moved on the sheet: SW1
