File: pcbs/backplane/cptrep_8500_backplane/cptrep_8500_backplane/cptrep_8500_backplane.kicad_pcb (KiCad board)
At the start: 2 copper layers, 147 x 185.4 mm, 5 parts, among them J1 Conn_02x50_Row_Letter_First, J2 Conn_02x50_Row_Letter_First, J3 Conn_02x50_Row_Letter_First, J4 Conn_02x50_Row_Letter_First, J5 Conn_02x50_Row_Letter_First

Commit message: "Update"
Parts:
- added C1: C_Small, Capacitor_SMD:C_0805_2012Metric_Pad1.18x1.45mm_HandSolder, F.Cu at (19.1, 42.6)
- added C2: C_Small, Capacitor_SMD:C_0805_2012Metric_Pad1.18x1.45mm_HandSolder, F.Cu at (19.1, 40.1)
- added D1: LED, LED_SMD:LED_0805_2012Metric_Pad1.15x1.40mm_HandSolder, F.Cu at (2.76, 50.5)
- added D2: LED, LED_SMD:LED_0805_2012Metric_Pad1.15x1.40mm_HandSolder, F.Cu at (2.76, 54.4)
- added D3: LED, LED_SMD:LED_0805_2012Metric_Pad1.15x1.40mm_HandSolder, F.Cu at (2.76, 62.0)
- added D4: LED, LED_SMD:LED_0805_2012Metric_Pad1.15x1.40mm_HandSolder, F.Cu at (2.76, 58.2)
- added D5: LED, LED_SMD:LED_0805_2012Metric_Pad1.15x1.40mm_HandSolder, F.Cu at (2.76, 65.8)
- added J10: Screw_Terminal_01x04, TerminalBlock_Phoenix:TerminalBlock_Phoenix_MKDS-1,5-4_1x04_P5.00mm_Horizontal, F.Cu at (8.64, 179.1)
- added J7: Screw_Terminal_01x04, TerminalBlock_Phoenix:TerminalBlock_Phoenix_MKDS-1,5-4_1x04_P5.00mm_Horizontal, F.Cu at (8.64, 114.5)
- added J8: Screw_Terminal_01x04, TerminalBlock_Phoenix:TerminalBlock_Phoenix_MKDS-1,5-4_1x04_P5.00mm_Horizontal, F.Cu at (8.64, 135.9)
- added J9: Screw_Terminal_01x04, TerminalBlock_Phoenix:TerminalBlock_Phoenix_MKDS-1,5-4_1x04_P5.00mm_Horizontal, F.Cu at (8.64, 157.2)
- added R1: 4k7, Resistor_SMD:R_0805_2012Metric_Pad1.20x1.40mm_HandSolder, F.Cu at (10.7, 50.5)
- added R2: 2k2, Resistor_SMD:R_0805_2012Metric_Pad1.20x1.40mm_HandSolder, F.Cu at (10.7, 54.4)
- added R3: 1k, Resistor_SMD:R_0805_2012Metric_Pad1.20x1.40mm_HandSolder, F.Cu at (10.7, 58.2)
- added R4: 2k2, Resistor_SMD:R_0805_2012Metric_Pad1.20x1.40mm_HandSolder, F.Cu at (10.7, 62.0)
- added R5: 1k, Resistor_SMD:R_0805_2012Metric_Pad1.20x1.40mm_HandSolder, F.Cu at (10.7, 65.8)
- added SW1: SW_Push, Button_Switch_THT:SW_PUSH_6mm, F.Cu at (199.2, 22.9)
- added U1: LM7905_TO220, Package_TO_SOT_THT:TO-220-3_Horizontal_TabDown, F.Cu at (16.5, 36.8)
- J1, J2, J3, J4, J5: value Conn_02x50_Row_Letter_First -> cpt-backplane_100; footprint Connector_Samtec_HLE_THT:Samtec_HLE-150-02-xx-DV-TE_2x50_P2.54mm_Horizontal -> ajm-cpt:cpt-8500-backplane-connector
- moved J2 129.5 mm to (98.8, 39.0), turned to 0 degrees
- moved J4 129.2 mm to (133.3, 39.0), turned to 0 degrees
- moved J1 126.8 mm to (64.3, 39.0), turned to 0 degrees
- moved J3 126.6 mm to (81.5, 39.0), turned to 0 degrees
- moved J5 126.1 mm to (116.1, 39.0), turned to 0 degrees
Connections:
- J1 pad 1: (no net) -> GND
- J1 pad 10: (no net) -> /CLEAR
- J1 pad 100: (no net) -> GND
- J1 pad 11: (no net) -> /RESET
- J1 pad 12: (no net) -> BP12
- J1 pad 13: (no net) -> READY
- J1 pad 14: (no net) -> /WAIT
- J1 pad 15: (no net) -> BP15
- J1 pad 16: (no net) -> BP16
- J1 pad 17: (no net) -> AUD
- J1 pad 18: (no net) -> BP18
- J1 pad 19: (no net) -> BP19
- J1 pad 2: (no net) -> GND
- J1 pad 20: (no net) -> /DB0
- J1 pad 21: (no net) -> /DB1
- J1 pad 22: (no net) -> /DB2
- J1 pad 23: (no net) -> /DB3
- J1 pad 24: (no net) -> /DB4
- J1 pad 25: (no net) -> /DB5
- J1 pad 26: (no net) -> /DB6
- J1 pad 27: (no net) -> /DB7
- J1 pad 28: (no net) -> /DB8
- J1 pad 29: (no net) -> /HLDAK
- J1 pad 3: (no net) -> GND
- J1 pad 30: (no net) -> /MEMRD
- J1 pad 31: (no net) -> /IORD
- J1 pad 32: (no net) -> /MEMWR
- J1 pad 33: (no net) -> /IOWR
- J1 pad 34: (no net) -> GND
- J1 pad 35: (no net) -> /BIN
- J1 pad 36: (no net) -> GND
- J1 pad 37: (no net) -> /BOUT
- J1 pad 38: (no net) -> GND
- J1 pad 39: (no net) -> BP39
- J1 pad 4: (no net) -> GND
- J1 pad 40: (no net) -> /A0
- J1 pad 41: (no net) -> /A1
- J1 pad 42: (no net) -> /A2
- J1 pad 43: (no net) -> /A3
- J1 pad 44: (no net) -> /A4
- J1 pad 45: (no net) -> /A5
- J1 pad 46: (no net) -> /A6
- J1 pad 47: (no net) -> /A7
- J1 pad 48: (no net) -> /A8
- J1 pad 49: (no net) -> /A9
- J1 pad 5: (no net) -> +24V
- J1 pad 50: (no net) -> /A10
- J1 pad 51: (no net) -> /A11
- J1 pad 52: (no net) -> /A12
- J1 pad 53: (no net) -> /A13
- J1 pad 54: (no net) -> /A14
- J1 pad 55: (no net) -> /A15
- J1 pad 56: (no net) -> /TC
- J1 pad 57: (no net) -> /REF
- J1 pad 58: (no net) -> /PE
- J1 pad 59: (no net) -> /BP59
- J1 pad 6: (no net) -> +24V
- J1 pad 60: (no net) -> /IO60
- J1 pad 61: (no net) -> /IO20
- J1 pad 62: (no net) -> /BP62
- J1 pad 63: (no net) -> /IO30
- J1 pad 64: (no net) -> /BP64
- J1 pad 65: (no net) -> /IO40
- J1 pad 66: (no net) -> /BP66
- J1 pad 67: (no net) -> /EOF
- J1 pad 68: (no net) -> /BP68
- J1 pad 69: (no net) -> /INT4
- J1 pad 7: (no net) -> +24V
- J1 pad 70: (no net) -> /BP70
- J1 pad 71: (no net) -> /INT3
- J1 pad 72: (no net) -> /INT1
- J1 pad 73: (no net) -> /DREQ0
- J1 pad 74: (no net) -> /DACK0
- J1 pad 75: (no net) -> /DREQ1
- J1 pad 76: (no net) -> /DACK1
- J1 pad 77: (no net) -> /DREQ2
- J1 pad 78: (no net) -> /DACK2
- J1 pad 79: (no net) -> /DREQ3
- J1 pad 8: (no net) -> +24V
- J1 pad 80: (no net) -> /DACK3
- J1 pad 81: (no net) -> PHI2
- J1 pad 82: (no net) -> GND
- J1 pad 83: (no net) -> /BP83
- J1 pad 84: (no net) -> GND
- J1 pad 85: (no net) -> /BP85
- J1 pad 86: (no net) -> GND
- J1 pad 87: (no net) -> -5V
- J1 pad 88: (no net) -> -5V
- J1 pad 89: (no net) -> -12V
- J1 pad 9: (no net) -> BP9
- J1 pad 90: (no net) -> -12V
- J1 pad 91: (no net) -> +12V
- J1 pad 92: (no net) -> +12V
- J1 pad 93: (no net) -> +5V
- J1 pad 94: (no net) -> +5V
- J1 pad 95: (no net) -> +5V
- J1 pad 96: (no net) -> +5V
- J1 pad 97: (no net) -> GND
- J1 pad 98: (no net) -> GND
- J1 pad 99: (no net) -> GND
- J2 pad 1: (no net) -> GND
- J2 pad 10: (no net) -> /CLEAR
- J2 pad 100: (no net) -> GND
- J2 pad 11: (no net) -> /RESET
- J2 pad 12: (no net) -> BP12
- J2 pad 13: (no net) -> READY
- J2 pad 14: (no net) -> /WAIT
- J2 pad 15: (no net) -> BP15
- J2 pad 16: (no net) -> BP16
- J2 pad 17: (no net) -> AUD
- J2 pad 18: (no net) -> BP18
- J2 pad 19: (no net) -> BP19
- J2 pad 2: (no net) -> GND
- J2 pad 20: (no net) -> /DB0
- J2 pad 21: (no net) -> /DB1
- J2 pad 22: (no net) -> /DB2
- J2 pad 23: (no net) -> /DB3
- J2 pad 24: (no net) -> /DB4
- J2 pad 25: (no net) -> /DB5
- J2 pad 26: (no net) -> /DB6
- J2 pad 27: (no net) -> /DB7
- J2 pad 28: (no net) -> /DB8
- J2 pad 29: (no net) -> /HLDAK
- J2 pad 3: (no net) -> GND
- J2 pad 30: (no net) -> /MEMRD
- J2 pad 31: (no net) -> /IORD
- J2 pad 32: (no net) -> /MEMWR
- J2 pad 33: (no net) -> /IOWR
- J2 pad 34: (no net) -> GND
- J2 pad 35: (no net) -> /BIN
- J2 pad 36: (no net) -> GND
- J2 pad 37: (no net) -> /BOUT
- J2 pad 38: (no net) -> GND
- J2 pad 39: (no net) -> BP39
- J2 pad 4: (no net) -> GND
- J2 pad 40: (no net) -> /A0
- J2 pad 41: (no net) -> /A1
- J2 pad 42: (no net) -> /A2
- J2 pad 43: (no net) -> /A3
- J2 pad 44: (no net) -> /A4
- J2 pad 45: (no net) -> /A5
- J2 pad 46: (no net) -> /A6
- J2 pad 47: (no net) -> /A7
- J2 pad 48: (no net) -> /A8
- J2 pad 49: (no net) -> /A9
- J2 pad 5: (no net) -> +24V
- J2 pad 50: (no net) -> /A10
- J2 pad 51: (no net) -> /A11
- J2 pad 52: (no net) -> /A12
- J2 pad 53: (no net) -> /A13
- J2 pad 54: (no net) -> /A14
- J2 pad 55: (no net) -> /A15
- J2 pad 56: (no net) -> /TC
- J2 pad 57: (no net) -> /REF
- J2 pad 58: (no net) -> /PE
- J2 pad 59: (no net) -> /BP59
- J2 pad 6: (no net) -> +24V
- J2 pad 60: (no net) -> /IO60
- J2 pad 61: (no net) -> /IO20
- J2 pad 62: (no net) -> /BP62
- J2 pad 63: (no net) -> /IO30
- J2 pad 64: (no net) -> /BP64
- J2 pad 65: (no net) -> /IO40
- J2 pad 66: (no net) -> /BP66
- J2 pad 67: (no net) -> /EOF
- J2 pad 68: (no net) -> /BP68
- J2 pad 69: (no net) -> /INT4
- J2 pad 7: (no net) -> +24V
- J2 pad 70: (no net) -> /BP70
- J2 pad 71: (no net) -> /INT3
- J2 pad 72: (no net) -> /INT1
- J2 pad 73: (no net) -> /DREQ0
- J2 pad 74: (no net) -> /DACK0
- J2 pad 75: (no net) -> /DREQ1
- J2 pad 76: (no net) -> /DACK1
- J2 pad 77: (no net) -> /DREQ2
- J2 pad 78: (no net) -> /DACK2
- J2 pad 79: (no net) -> /DREQ3
- J2 pad 8: (no net) -> +24V
- J2 pad 80: (no net) -> /DACK3
- J2 pad 81: (no net) -> PHI2
- J2 pad 82: (no net) -> GND
- J2 pad 83: (no net) -> /BP83
- J2 pad 84: (no net) -> GND
- J2 pad 85: (no net) -> /BP85
- J2 pad 86: (no net) -> GND
- J2 pad 87: (no net) -> -5V
- J2 pad 88: (no net) -> -5V
- J2 pad 89: (no net) -> -12V
- J2 pad 9: (no net) -> BP9
- J2 pad 90: (no net) -> -12V
- J2 pad 91: (no net) -> +12V
- J2 pad 92: (no net) -> +12V
- J2 pad 93: (no net) -> +5V
- J2 pad 94: (no net) -> +5V
- J2 pad 95: (no net) -> +5V
- J2 pad 96: (no net) -> +5V
- J2 pad 97: (no net) -> GND
- J2 pad 98: (no net) -> GND
- J2 pad 99: (no net) -> GND
- J3 pad 1: (no net) -> GND
- J3 pad 10: (no net) -> /CLEAR
- J3 pad 100: (no net) -> GND
- J3 pad 11: (no net) -> /RESET
- J3 pad 12: (no net) -> BP12
- J3 pad 13: (no net) -> READY
- J3 pad 14: (no net) -> /WAIT
- J3 pad 15: (no net) -> BP15
- J3 pad 16: (no net) -> BP16
- J3 pad 17: (no net) -> AUD
- J3 pad 18: (no net) -> BP18
- J3 pad 19: (no net) -> BP19
- J3 pad 2: (no net) -> GND
- J3 pad 20: (no net) -> /DB0
- J3 pad 21: (no net) -> /DB1
- J3 pad 22: (no net) -> /DB2
- J3 pad 23: (no net) -> /DB3
- J3 pad 24: (no net) -> /DB4
- J3 pad 25: (no net) -> /DB5
- J3 pad 26: (no net) -> /DB6
- J3 pad 27: (no net) -> /DB7
- J3 pad 28: (no net) -> /DB8
- J3 pad 29: (no net) -> /HLDAK
- J3 pad 3: (no net) -> GND
- J3 pad 30: (no net) -> /MEMRD
- J3 pad 31: (no net) -> /IORD
- J3 pad 32: (no net) -> /MEMWR
- J3 pad 33: (no net) -> /IOWR
- J3 pad 34: (no net) -> GND
- J3 pad 35: (no net) -> /BIN
- J3 pad 36: (no net) -> GND
- J3 pad 37: (no net) -> /BOUT
- J3 pad 38: (no net) -> GND
- J3 pad 39: (no net) -> BP39
- J3 pad 4: (no net) -> GND
- J3 pad 40: (no net) -> /A0
- J3 pad 41: (no net) -> /A1
- J3 pad 42: (no net) -> /A2
- J3 pad 43: (no net) -> /A3
- J3 pad 44: (no net) -> /A4
- J3 pad 45: (no net) -> /A5
- J3 pad 46: (no net) -> /A6
- J3 pad 47: (no net) -> /A7
- J3 pad 48: (no net) -> /A8
- J3 pad 49: (no net) -> /A9
- J3 pad 5: (no net) -> +24V
- J3 pad 50: (no net) -> /A10
- J3 pad 51: (no net) -> /A11
- J3 pad 52: (no net) -> /A12
- J3 pad 53: (no net) -> /A13
- J3 pad 54: (no net) -> /A14
- J3 pad 55: (no net) -> /A15
- J3 pad 56: (no net) -> /TC
- J3 pad 57: (no net) -> /REF
- J3 pad 58: (no net) -> /PE
- J3 pad 59: (no net) -> /BP59
- J3 pad 6: (no net) -> +24V
- J3 pad 60: (no net) -> /IO60
- J3 pad 61: (no net) -> /IO20
- J3 pad 62: (no net) -> /BP62
- J3 pad 63: (no net) -> /IO30
- J3 pad 64: (no net) -> /BP64
- J3 pad 65: (no net) -> /IO40
- J3 pad 66: (no net) -> /BP66
- J3 pad 67: (no net) -> /EOF
- J3 pad 68: (no net) -> /BP68
- J3 pad 69: (no net) -> /INT4
- J3 pad 7: (no net) -> +24V
- J3 pad 70: (no net) -> /BP70
- J3 pad 71: (no net) -> /INT3
- J3 pad 72: (no net) -> /INT1
- J3 pad 73: (no net) -> /DREQ0
- J3 pad 74: (no net) -> /DACK0
- J3 pad 75: (no net) -> /DREQ1
- J3 pad 76: (no net) -> /DACK1
- J3 pad 77: (no net) -> /DREQ2
- J3 pad 78: (no net) -> /DACK2
- J3 pad 79: (no net) -> /DREQ3
- J3 pad 8: (no net) -> +24V
- J3 pad 80: (no net) -> /DACK3
- J3 pad 81: (no net) -> PHI2
- J3 pad 82: (no net) -> GND
- J3 pad 83: (no net) -> /BP83
- J3 pad 84: (no net) -> GND
- J3 pad 85: (no net) -> /BP85
- J3 pad 86: (no net) -> GND
- J3 pad 87: (no net) -> -5V
- J3 pad 88: (no net) -> -5V
- J3 pad 89: (no net) -> -12V
- J3 pad 9: (no net) -> BP9
- J3 pad 90: (no net) -> -12V
- J3 pad 91: (no net) -> +12V
- J3 pad 92: (no net) -> +12V
- J3 pad 93: (no net) -> +5V
- J3 pad 94: (no net) -> +5V
- J3 pad 95: (no net) -> +5V
- J3 pad 96: (no net) -> +5V
- J3 pad 97: (no net) -> GND
- J3 pad 98: (no net) -> GND
- J3 pad 99: (no net) -> GND
- J4 pad 1: (no net) -> GND
- J4 pad 10: (no net) -> /CLEAR
- J4 pad 100: (no net) -> GND
- J4 pad 11: (no net) -> /RESET
- J4 pad 12: (no net) -> BP12
- J4 pad 13: (no net) -> READY
- J4 pad 14: (no net) -> /WAIT
- J4 pad 15: (no net) -> BP15
- J4 pad 16: (no net) -> BP16
- J4 pad 17: (no net) -> AUD
- J4 pad 18: (no net) -> BP18
- J4 pad 19: (no net) -> BP19
- J4 pad 2: (no net) -> GND
- J4 pad 20: (no net) -> /DB0
- J4 pad 21: (no net) -> /DB1
- J4 pad 22: (no net) -> /DB2
- J4 pad 23: (no net) -> /DB3
- J4 pad 24: (no net) -> /DB4
- J4 pad 25: (no net) -> /DB5
- J4 pad 26: (no net) -> /DB6
- J4 pad 27: (no net) -> /DB7
- J4 pad 28: (no net) -> /DB8
- J4 pad 29: (no net) -> /HLDAK
- J4 pad 3: (no net) -> GND
- J4 pad 30: (no net) -> /MEMRD
- J4 pad 31: (no net) -> /IORD
- J4 pad 32: (no net) -> /MEMWR
- J4 pad 33: (no net) -> /IOWR
- J4 pad 34: (no net) -> GND
- J4 pad 35: (no net) -> /BIN
- J4 pad 36: (no net) -> GND
- J4 pad 37: (no net) -> /BOUT
- J4 pad 38: (no net) -> GND
- J4 pad 39: (no net) -> BP39
- J4 pad 4: (no net) -> GND
- J4 pad 40: (no net) -> /A0
- J4 pad 41: (no net) -> /A1
- J4 pad 42: (no net) -> /A2
- J4 pad 43: (no net) -> /A3
- J4 pad 44: (no net) -> /A4
- J4 pad 45: (no net) -> /A5
- J4 pad 46: (no net) -> /A6
- J4 pad 47: (no net) -> /A7
- J4 pad 48: (no net) -> /A8
- J4 pad 49: (no net) -> /A9
- J4 pad 5: (no net) -> +24V
- J4 pad 50: (no net) -> /A10
- J4 pad 51: (no net) -> /A11
- J4 pad 52: (no net) -> /A12
- J4 pad 53: (no net) -> /A13
- J4 pad 54: (no net) -> /A14
- J4 pad 55: (no net) -> /A15
- J4 pad 56: (no net) -> /TC
- J4 pad 57: (no net) -> /REF
- J4 pad 58: (no net) -> /PE
- J4 pad 59: (no net) -> /BP59
- J4 pad 6: (no net) -> +24V
- J4 pad 60: (no net) -> /IO60
- J4 pad 61: (no net) -> /IO20
- J4 pad 62: (no net) -> /BP62
- J4 pad 63: (no net) -> /IO30
- J4 pad 64: (no net) -> /BP64
- J4 pad 65: (no net) -> /IO40
- J4 pad 66: (no net) -> /BP66
- J4 pad 67: (no net) -> /EOF
- J4 pad 68: (no net) -> /BP68
- J4 pad 69: (no net) -> /INT4
- J4 pad 7: (no net) -> +24V
- J4 pad 70: (no net) -> /BP70
- J4 pad 71: (no net) -> /INT3
- J4 pad 72: (no net) -> /INT1
- J4 pad 73: (no net) -> /DREQ0
- J4 pad 74: (no net) -> /DACK0
- J4 pad 75: (no net) -> /DREQ1
- J4 pad 76: (no net) -> /DACK1
- J4 pad 77: (no net) -> /DREQ2
- J4 pad 78: (no net) -> /DACK2
- J4 pad 79: (no net) -> /DREQ3
- J4 pad 8: (no net) -> +24V
- J4 pad 80: (no net) -> /DACK3
- J4 pad 81: (no net) -> PHI2
- J4 pad 82: (no net) -> GND
- J4 pad 83: (no net) -> /BP83
- J4 pad 84: (no net) -> GND
- J4 pad 85: (no net) -> /BP85
- J4 pad 86: (no net) -> GND
- J4 pad 87: (no net) -> -5V
- J4 pad 88: (no net) -> -5V
- J4 pad 89: (no net) -> -12V
- J4 pad 9: (no net) -> BP9
- J4 pad 90: (no net) -> -12V
- J4 pad 91: (no net) -> +12V
- J4 pad 92: (no net) -> +12V
- J4 pad 93: (no net) -> +5V
- J4 pad 94: (no net) -> +5V
- J4 pad 95: (no net) -> +5V
- J4 pad 96: (no net) -> +5V
- J4 pad 97: (no net) -> GND
- J4 pad 98: (no net) -> GND
- J4 pad 99: (no net) -> GND
- J5 pad 1: (no net) -> GND
- J5 pad 10: (no net) -> /CLEAR
- J5 pad 100: (no net) -> GND
- J5 pad 11: (no net) -> /RESET
- J5 pad 12: (no net) -> BP12
- J5 pad 13: (no net) -> READY
- J5 pad 14: (no net) -> /WAIT
- J5 pad 15: (no net) -> BP15
- J5 pad 16: (no net) -> BP16
- J5 pad 17: (no net) -> AUD
- J5 pad 18: (no net) -> BP18
- J5 pad 19: (no net) -> BP19
- J5 pad 2: (no net) -> GND
- J5 pad 20: (no net) -> /DB0
- J5 pad 21: (no net) -> /DB1
- J5 pad 22: (no net) -> /DB2
- J5 pad 23: (no net) -> /DB3
- J5 pad 24: (no net) -> /DB4
- J5 pad 25: (no net) -> /DB5
- J5 pad 26: (no net) -> /DB6
- J5 pad 27: (no net) -> /DB7
- J5 pad 28: (no net) -> /DB8
- J5 pad 29: (no net) -> /HLDAK
- J5 pad 3: (no net) -> GND
- J5 pad 30: (no net) -> /MEMRD
- J5 pad 31: (no net) -> /IORD
- J5 pad 32: (no net) -> /MEMWR
- J5 pad 33: (no net) -> /IOWR
- J5 pad 34: (no net) -> GND
- J5 pad 35: (no net) -> /BIN
- J5 pad 36: (no net) -> GND
- J5 pad 37: (no net) -> /BOUT
- J5 pad 38: (no net) -> GND
- J5 pad 39: (no net) -> BP39
- J5 pad 4: (no net) -> GND
- J5 pad 40: (no net) -> /A0
- J5 pad 41: (no net) -> /A1
- J5 pad 42: (no net) -> /A2
- J5 pad 43: (no net) -> /A3
- J5 pad 44: (no net) -> /A4
- J5 pad 45: (no net) -> /A5
- J5 pad 46: (no net) -> /A6
- J5 pad 47: (no net) -> /A7
- J5 pad 48: (no net) -> /A8
- J5 pad 49: (no net) -> /A9
- J5 pad 5: (no net) -> +24V
- J5 pad 50: (no net) -> /A10
- J5 pad 51: (no net) -> /A11
- J5 pad 52: (no net) -> /A12
- J5 pad 53: (no net) -> /A13
- J5 pad 54: (no net) -> /A14
- J5 pad 55: (no net) -> /A15
- J5 pad 56: (no net) -> /TC
- J5 pad 57: (no net) -> /REF
- J5 pad 58: (no net) -> /PE
- J5 pad 59: (no net) -> /BP59
- J5 pad 6: (no net) -> +24V
- J5 pad 60: (no net) -> /IO60
- J5 pad 61: (no net) -> /IO20
- J5 pad 62: (no net) -> /BP62
- J5 pad 63: (no net) -> /IO30
- J5 pad 64: (no net) -> /BP64
- J5 pad 65: (no net) -> /IO40
- J5 pad 66: (no net) -> /BP66
- J5 pad 67: (no net) -> /EOF
- J5 pad 68: (no net) -> /BP68
- J5 pad 69: (no net) -> /INT4
- J5 pad 7: (no net) -> +24V
- J5 pad 70: (no net) -> /BP70
- J5 pad 71: (no net) -> /INT3
- J5 pad 72: (no net) -> /INT1
- J5 pad 73: (no net) -> /DREQ0
- J5 pad 74: (no net) -> /DACK0
- J5 pad 75: (no net) -> /DREQ1
- J5 pad 76: (no net) -> /DACK1
- J5 pad 77: (no net) -> /DREQ2
- J5 pad 78: (no net) -> /DACK2
- J5 pad 79: (no net) -> /DREQ3
- J5 pad 8: (no net) -> +24V
- J5 pad 80: (no net) -> /DACK3
- J5 pad 81: (no net) -> PHI2
- J5 pad 82: (no net) -> GND
- J5 pad 83: (no net) -> /BP83
- J5 pad 84: (no net) -> GND
- J5 pad 85: (no net) -> /BP85
- J5 pad 86: (no net) -> GND
- J5 pad 87: (no net) -> -5V
- J5 pad 88: (no net) -> -5V
- J5 pad 89: (no net) -> -12V
- J5 pad 9: (no net) -> BP9
- J5 pad 90: (no net) -> -12V
- J5 pad 91: (no net) -> +12V
- J5 pad 92: (no net) -> +12V
- J5 pad 93: (no net) -> +5V
- J5 pad 94: (no net) -> +5V
- J5 pad 95: (no net) -> +5V
- J5 pad 96: (no net) -> +5V
- J5 pad 97: (no net) -> GND
- J5 pad 98: (no net) -> GND
- J5 pad 99: (no net) -> GND
Routing:
- net (no net): track 215.0 -> 0.00 mm
Other:
- board size 147 x 185.4 mm -> 146 x 196.2 mm

Commit message: "Update"
Parts:
- moved SW1 194.6 mm to (12.1, 76.4), turned to 180 degrees
- moved J10 72.2 mm to (9.91, 106.8)
- moved J8 18.2 mm to (9.98, 154.0)
- moved J9 18.2 mm to (9.98, 175.4)
- moved J7 18.2 mm to (9.98, 132.7)
- moved D1 1.31 mm to (3.70, 51.5)
- moved D2 1.31 mm to (3.70, 55.3)
- moved D3 1.31 mm to (3.70, 62.9)
- moved D4 1.31 mm to (3.70, 59.1)
- moved D5 1.31 mm to (3.70, 66.7), turned to 0 degrees
- moved R1 1.31 mm to (11.6, 51.5), turned to 180 degrees
- moved R2 1.31 mm to (11.6, 55.3), turned to 180 degrees
- moved R3 1.31 mm to (11.6, 59.1), turned to 180 degrees
- moved R4 1.31 mm to (11.6, 62.9), turned to 180 degrees
- moved R5 1.31 mm to (11.6, 66.7), turned to 180 degrees
Routing:
- net GND: track 0.00 -> 1807.0 mm
- net +5V: track 0.00 -> 1385.8 mm, vias 0 -> 1
- net -12V: track 0.00 -> 313.1 mm, vias 0 -> 3
- net -5V: track 0.00 -> 301.5 mm, vias 0 -> 3
- net +12V: track 0.00 -> 280.1 mm, vias 0 -> 2
- net +24V: track 0.00 -> 220.9 mm, vias 0 -> 1
- net AUD: track 0.00 -> 195.2 mm
- net /CLEAR: track 0.00 -> 193.0 mm
- net /BP85: track 0.00 -> 123.8 mm
- net /BP83: track 0.00 -> 122.6 mm
- net /DREQ3: track 0.00 -> 73.4 mm
- net /IO30: track 0.00 -> 73.4 mm
- net /EOF: track 0.00 -> 73.4 mm
- net BP39: track 0.00 -> 73.4 mm
- net /RESET: track 0.00 -> 73.4 mm
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- added copper zone on B.Cu, net (none)
- added copper zone on F.Cu, net GND
Other:
- outline, holes or cut-outs redrawn
- board text added: "+12V"
- board text added: "+24V"
- board text added: "+5V"
- board text added: "-12V"
- board text added: "-5V"
- board text added: "1 GND"
- board text added: "10 GND"
- board text added: "11 GND"
- board text added: "12 +5V"
- board text added: "2 /CLEAR"
- board text added: "3 AUD"
- board text added: "4 BP83"
- board text added: "5 BP85"
- board text added: "6 GND"
- board text added: "7 GND"
- board text added: "8 GND"
- board text added: "9 +12V"

Commit message: "Update"
Connections:
- J10 pad 1: unconnected-(J10-Pin_1-Pad1) -> +24V
- J10 pad 4: unconnected-(J10-Pin_4-Pad4) -> GND
Routing:
- net (no net): track 0.00 -> 164.1 mm, vias 10 -> 13
- net +24V: track 220.9 -> 283.2 mm, vias 1 -> 2
- net GND: track 1807.0 -> 1822.7 mm
- net +5V: track 1385.8 -> 1394.5 mm, vias 1 -> 2
Other:
- board text added: "1 +24V"
- board text added: "4 GND"
- board text added: "CPT Replica Backplane V1.0 Mar 2026 menadue@gmail.com"

Commit message: "Update"
Parts:
- added J6: Conn_01x02_Pin, Connector_PinSocket_2.54mm:PinSocket_1x02_P2.54mm_Vertical, F.Cu at (4.33, 89.5)
- added R6: 27R, Resistor_SMD:R_0805_2012Metric_Pad1.20x1.40mm_HandSolder, F.Cu at (4.20, 82.5)
Connections:
- SW1 pad 1: unconnected-(SW1-Pad1) -> Net-(R6-Pad2)
- SW1 pad 2: unconnected-(SW1-Pad2) -> /CLEAR
Routing:
- net /CLEAR: track 193.0 -> 281.0 mm
- net AUD: track 195.2 -> 250.8 mm
- net GND: track 1822.7 -> 1876.3 mm, vias 0 -> 2
- net (no net): track 164.1 -> 145.6 mm, vias 13 -> 12
- net Net-(R6-Pad2): track 0.00 -> 18.3 mm
- net +5V: track 1394.5 -> 1387.8 mm, vias 2 -> 1
Other:
- board text added: "Audio"

Commit message: "Update"
Other:
- board text added: "RESET"
Changed lines of the file:
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@@
+		)
+	)
+	(gr_text "RESET"
+		(at 15 74.9 0)
+		(layer "F.SilkS")
+		(effects
+			(font
+				(size 1 1)
+				(thickness 0.1)
+			)
+			(justify left bottom)
 		)
 	)
