File: pcbs/diagcard/cptrep-diag-card/cpt-connector.kicad_sch (KiCad schematic)
At the start: 56 parts, among them J2 cpt-backplane_100

Commit message: "Update"
Parts:
- J2: footprint (none) -> ajm-cpt:cpt-card-edge-100
Changed lines of the file:
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@@
 			)
 		)
-		(property "Footprint" ""
+		(property "Footprint" "ajm-cpt:cpt-card-edge-100"
 			(at 146.05 86.995 0)
 			(effects

Commit message: "Update"
Connections:
- net GND: now also J2.1 (GND), J2.2 (GND), J2.3 (GND), J2.4 (GND)
Changed lines of the file:
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@@
 		)
 	)
+	(junction
+		(at 160.655 28.575)
+		(diameter 0)
+		(color 0 0 0 0)
+	)
+	(junction
+		(at 112.395 28.575)
+		(diameter 0)
+		(color 0 0 0 0)
+	)
 	(wire
 		(pts
@@
 	(wire
 		(pts
+			(xy 153.67 26.035) (xy 160.655 26.035)
+		)
+		(stroke
+			(width 0)
+			(type default)
+		)
+	)
+	(wire
+		(pts
 			(xy 73.025 125.095) (xy 119.38 125.095)
 		)
@@
 	(wire
 		(pts
+			(xy 160.655 28.575) (xy 160.655 32.385)
+		)
+		(stroke
+			(width 0)
+			(type default)
+		)
+	)
+	(wire
+		(pts
 			(xy 202.565 79.375) (xy 153.67 79.375)
 		)
@@
 	(wire
 		(pts
+			(xy 112.395 28.575) (xy 112.395 32.385)
+		)
+		(stroke
+			(width 0)
+			(type default)
+		)
+	)
+	(wire
+		(pts
 			(xy 73.025 97.155) (xy 119.38 97.155)
 		)
@@
 	(wire
 		(pts
+			(xy 119.38 28.575) (xy 112.395 28.575)
+		)
+		(stroke
+			(width 0)
+			(type default)
+		)
+	)
+	(wire
+		(pts
 			(xy 216.535 74.295) (xy 207.645 74.295)
 		)
@@
 	(wire
 		(pts
+			(xy 160.655 26.035) (xy 160.655 28.575)
+		)
+		(stroke
+			(width 0)
+			(type default)
+		)
+	)
+	(wire
+		(pts
 			(xy 59.055 97.155) (xy 67.945 97.155)
 		)
@@
 	(wire
 		(pts
+			(xy 153.67 28.575) (xy 160.655 28.575)
+		)
+		(stroke
+			(width 0)
+			(type default)
+		)
+	)
+	(wire
+		(pts
+			(xy 112.395 26.035) (xy 112.395 28.575)
+		)
+		(stroke
+			(width 0)
+			(type default)
+		)
+	)
+	(wire
+		(pts
 			(xy 59.055 102.235) (xy 67.945 102.235)
 		)
@@
 	(wire
 		(pts
+			(xy 119.38 26.035) (xy 112.395 26.035)
+		)
+		(stroke
+			(width 0)
+			(type default)
+		)
+	)
+	(wire
+		(pts
 			(xy 216.535 76.835) (xy 207.645 76.835)
 		)
@@
 	)
 	(symbol
+		(lib_id "pico-9000-pack-rescue:GND-power")
+		(at 112.395 32.385 0)
+		(unit 1)
+		(exclude_from_sim no)
+		(in_bom yes)
+		(on_board yes)
+		(dnp no)
+		(property "Reference" "#PWR035"
+			(at 112.395 38.735 0)
+			(effects
+				(font
+					(size 1.27 1.27)
+				)
+				(hide yes)
+			)
+		)
+		(property "Value" "GND"
+			(at 112.522 36.7792 0)
+			(effects
+				(font
+					(size 1.27 1.27)
+				)
+			)
+		)
+		(property "Footprint" ""
+			(at 112.395 32.385 0)
+			(effects
+				(font
+					(size 1.27 1.27)
+				)
+				(hide yes)
+			)
+		)
+		(property "Datasheet" ""
+			(at 112.395 32.385 0)
+			(effects
+				(font
+					(size 1.27 1.27)
+				)
+				(hide yes)
+			)
+		)
+		(property "Description" ""
+			(at 112.395 32.385 0)
+			(effects
+				(font
+					(size 1.27 1.27)
+				)
+				(hide yes)
+			)
+		)
+		(pin "1"
+		)
+		(instances
+			(project "cptrep-diag-card"
+				(path "/75f9f2a9-074b-4f58-a7a7-2a17dd71988c/233374be-d93d-42b3-b222-4739a83f5cdd"
+					(reference "#PWR035")
+					(unit 1)
+				)
+			)
+		)
+	)
+	(symbol
 		(lib_id "Device:R_Small")
 		(at 205.105 125.095 270)
@@
 					(unit 1)
 				)
+			)
+		)
+	)
+	(symbol
+		(lib_id "pico-9000-pack-rescue:GND-power")
+		(at 160.655 32.385 0)
+		(mirror y)
+		(unit 1)
+		(exclude_from_sim no)
+		(in_bom yes)
+		(on_board yes)
+		(dnp no)
+		(property "Reference" "#PWR034"
+			(at 160.655 38.735 0)
+			(effects
+				(font
+					(size 1.27 1.27)
+				)
+				(hide yes)
+			)
+		)
+		(property "Value" "GND"
+			(at 160.528 36.7792 0)
+			(effects
+				(font
+					(size 1.27 1.27)
+				)
+			)
+		)
+		(property "Footprint" ""
+			(at 160.655 32.385 0)
+			(effects
+				(font
+					(size 1.27 1.27)
+				)
+				(hide yes)
+			)
+		)
+		(property "Datasheet" ""
+			(at 160.655 32.385 0)
+			(effects
+				(font
+					(size 1.27 1.27)
+				)
+				(hide yes)
+			)
+		)
+		(property "Description" ""
+			(at 160.655 32.385 0)
+			(effects
+				(font
+					(size 1.27 1.27)
+				)
+				(hide yes)
+			)
+		)
+		(pin "1"
+		)
+		(instances
+			(project "cptrep-diag-card"
+				(path "/75f9f2a9-074b-4f58-a7a7-2a17dd71988c/233374be-d93d-42b3-b222-4739a83f5cdd"
+					(reference "#PWR034")
+					(unit 1)
+				)
