File: pcbs/diagcard/cptrep-diag-card/cptrep-diag-card.kicad_sch (KiCad schematic)
At the start: 0 parts

Commit message: "Update"
Parts:
- added D1: D_Schottky, Diode_SMD:D_SOD-123, symbol Device:D_Schottky
- added EXT1, EXT2: NA(HN2x20), Connector_PinSocket_2.54mm:PinSocket_2x20_P2.54mm_Vertical, symbol OLIMEX_Connectors:BH40S
- added J1: Conn_02x06_Counter_Clockwise, symbol Connector_Generic:Conn_02x06_Counter_Clockwise
- added J3, J4, J5, J6, J7: Conn_02x04_Counter_Clockwise, Connector_PinHeader_2.54mm:PinHeader_2x04_P2.54mm_Vertical, symbol Connector_Generic:Conn_02x04_Counter_Clockwise
- added XS1: 502p_SD_ebay-uSD-push_push_SMD, ajm-acorn:Conn_uSDcard, symbol pico-9000-pack-rescue:502p_SD_ebay-uSD-push_push_SMD-pak_breakout
Connections:
- new net +3.3V: EXT1.1, EXT1.2, EXT1.21, EXT1.22, EXT2.1, EXT2.21, EXT2.22, EXT2.8, XS1.4 (Vdd)
- new net +5V: D1.2 (A)
- new net 3V3_EN: EXT2.12
- new net ADC_VREF: EXT2.14
- new net BIN: J5.7 (Pin_7)
- new net BOOTSEL#: EXT2.20
- new net BOUT: J5.8 (Pin_8)
- new net DACK0: J4.6 (Pin_6)
- new net DACK1: J4.5 (Pin_5)
- new net DACK2: J3.6 (Pin_6)
- new net DACK3: J3.5 (Pin_5)
- new net DREQ0: J4.8 (Pin_8)
- new net DREQ1: J4.7 (Pin_7)
- new net DREQ2: J3.8 (Pin_8)
- new net DREQ3: J3.7 (Pin_7)
- new net EOF: J5.5 (Pin_5)
- new net GND: EXT1.19, EXT1.20, EXT1.39, EXT1.40, EXT2.10, EXT2.16, EXT2.19, EXT2.39, EXT2.40, EXT2.6, XS1.6 (GND)
- new net GPIO0: EXT1.4
- new net GPIO1: EXT1.6
- new net GPIO14: EXT1.36, J3.1 (Pin_1), J4.1 (Pin_1), J5.1 (Pin_1), J6.1 (Pin_1), J7.1 (Pin_1)
- new net GPIO15: EXT1.38, J3.2 (Pin_2), J4.2 (Pin_2), J5.2 (Pin_2), J6.2 (Pin_2), J7.2 (Pin_2)
- new net GPIO16: EXT1.3, J1.1 (Pin_1)
- new net GPIO17: EXT1.5, J3.3 (Pin_3), J4.3 (Pin_3), J5.3 (Pin_3), J6.3 (Pin_3), J7.3 (Pin_3)
- new net GPIO18: EXT1.7, J1.2 (Pin_2)
- new net GPIO19: EXT1.9, J1.3 (Pin_3)
- new net GPIO2: EXT1.8
- new net GPIO20: EXT1.11, J1.4 (Pin_4)
- new net GPIO21: EXT1.13, J1.5 (Pin_5)
- new net GPIO22: EXT1.15, J1.6 (Pin_6)
- new net GPIO26: EXT1.27, J4.4 (Pin_4), J5.4 (Pin_4), J6.4 (Pin_4), J7.4 (Pin_4)
- new net GPIO3: EXT1.10
- new net GPIO32: EXT2.3
- new net GPIO33: EXT2.5
- new net GPIO34: EXT2.7
- new net GPIO35: EXT2.9
- new net GPIO36: EXT2.11
- new net GPIO37: EXT2.13
- new net GPIO38: EXT2.15
- new net GPIO39: EXT2.17
- new net GPIO4: EXT1.12
- new net GPIO40: EXT2.23
- new net GPIO41: EXT2.25
- new net GPIO42: EXT2.27
- new net GPIO43: EXT2.29
- new net GPIO44: EXT2.31
- new net GPIO45: EXT2.33
- new net GPIO46: EXT2.35
- new net GPIO47: EXT2.37
- new net GPIO5: EXT1.14
- new net GPIO6: EXT1.16
- new net GPIO7: EXT1.18
- new net GPIO8: EXT1.24
- new net HLDACK: J6.8 (Pin_8)
- new net INT1: EXT1.25
- new net INT3: EXT1.23
- new net INT4: EXT1.17
- new net IO20: EXT1.37
- new net IO30: EXT1.35
- new net IO40: EXT1.33
- new net IO60: EXT1.31
- new net IORD: EXT1.30
- new net IOWR: EXT1.32
- new net MEMRD: EXT1.28
- new net MEMWR: EXT1.26
- new net MISO_DO: J1.12 (Pin_12), XS1.7 (DO/DAT0)
- new net MOSI_DI: J1.10 (Pin_10), XS1.3 (DI/CMD)
- new net PARITYERR: EXT1.29
- new net PHI2: EXT1.34
- new net QSPI_CLK: EXT2.32
- new net QSPI_CSn: EXT2.34
- new net QSPI_SD0: EXT2.24
- new net QSPI_SD1: EXT2.26
- new net QSPI_SD2: EXT2.28
- new net QSPI_SD3: EXT2.30
- new net READY: J6.6 (Pin_6)
- new net REF: J7.8 (Pin_8)
- new net RESET: J6.7 (Pin_7)
- new net RUN: EXT2.18
- new net SD_CLK: J1.11 (Pin_11), XS1.5 (CLK)
- new net SD_DAT1: J1.9 (Pin_9), XS1.8 (DAT1)
- new net SD_DAT2: J1.8 (Pin_8), XS1.1 (DAT2)
- new net SD_SS: J1.7 (Pin_7), XS1.2 (CS/DAT3)
- new net SWCLK: EXT2.38
- new net SWDIO: EXT2.36
- new net TC: J5.6 (Pin_6)
- new net VBUS: EXT2.2
- new net VSYS: D1.1 (K), EXT2.4
- new net WAIT: J6.5 (Pin_5)
Other:
- added sheet Connector (cpt-connector.kicad_sch)
- added sheet leds (leds.kicad_sch)
- note added: "GPIO0-7 D0-D7"
- note added: "GPIO32-47 A0-A15"

Commit message: "Update"
Parts:
- removed J1: Conn_02x06_Counter_Clockwise, symbol Connector_Generic:Conn_02x06_Counter_Clockwise
- added J10: Conn_02x06_Odd_Even, Connector_PinHeader_2.54mm:PinHeader_2x06_P2.54mm_Vertical, symbol Connector_Generic:Conn_02x06_Odd_Even
- XS1: footprint ajm-acorn:Conn_uSDcard -> ajm-sdcard:Conn_uSDcard
Connections:
- net GPIO16: now also J10.1 (Pin_1)
- net GPIO18: now also J10.3 (Pin_3)
- net GPIO19: now also J10.5 (Pin_5)
- net GPIO20: now also J10.7 (Pin_7)
- net GPIO21: now also J10.9 (Pin_9)
- net GPIO22: now also J10.11 (Pin_11)
- net MISO_DO: now also J10.2 (Pin_2)
- net MOSI_DI: now also J10.6 (Pin_6)
- net SD_CLK: now also J10.4 (Pin_4)
- net SD_DAT1: now also J10.8 (Pin_8)
- net SD_DAT2: now also J10.10 (Pin_10)
- net SD_SS: now also J10.12 (Pin_12)
Changed lines of the file:
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@@
+	)
+	(symbol
+		(lib_id "Connector_Generic:Conn_02x06_Odd_Even")
+		(at 151.13 45.085 0)
+		(unit 1)
+		(exclude_from_sim no)
+		(in_bom yes)
+		(on_board yes)
+		(dnp no)
+		(fields_autoplaced yes)
+		(property "Reference" "J10"
+			(at 152.4 34.29 0)
+			(effects
+				(font
+					(size 1.27 1.27)
+				)
+			)
+		)
+		(property "Value" "Conn_02x06_Odd_Even"
+			(at 152.4 36.83 0)
+			(effects
+				(font
+					(size 1.27 1.27)
+				)
+			)
+		)
+		(property "Footprint" "Connector_PinHeader_2.54mm:PinHeader_2x06_P2.54mm_Vertical"
+			(at 151.13 45.085 0)
+			(effects
+				(font
+					(size 1.27 1.27)
+				)
+				(hide yes)
+			)
+		)
+		(property "Datasheet" "~"
+			(at 151.13 45.085 0)
+			(effects
+				(font
+					(size 1.27 1.27)
+				)
+				(hide yes)
+			)
+		)
+		(property "Description" "Generic connector, double row, 02x06, odd/even pin numbering scheme (row 1 odd numbers, row 2 even numbers), script generated (kicad-library-utils/schlib/autogen/connector/)"
+			(at 151.13 45.085 0)
+			(effects
+				(font
+					(size 1.27 1.27)
+				)
+				(hide yes)
+			)
+		)
+		(pin "7"
+		)
+		(pin "6"
+		)
+		(pin "10"
+		)
+		(pin "9"
+		)
+		(pin "5"
+		)
+		(pin "12"
+		)
+		(pin "11"
+		)
+		(pin "2"
+		)
+		(pin "3"
+		)
+		(pin "1"
+		)
+		(pin "8"
+		)
+		(pin "4"
+		)
+		(instances
+			(project ""
+				(path "/75f9f2a9-074b-4f58-a7a7-2a17dd71988c"
+					(reference "J10")
+					(unit 1)
+				)
+			)
+		)
 	)
 	(symbol
@@
 	)
 	(symbol
-		(lib_id "Connector_Generic:Conn_02x06_Counter_Clockwise")
-		(at 151.13 45.085 0)
-		(unit 1)
-		(exclude_from_sim no)
-		(in_bom yes)
-		(on_board yes)
-		(dnp no)
-		(fields_autoplaced yes)
-		(property "Reference" "J1"
-			(at 152.4 33.655 0)
-			(effects
-				(font
-					(size 1.27 1.27)
-				)
-			)
-		)
-		(property "Value" "Conn_02x06_Counter_Clockwise"
-			(at 152.4 36.195 0)
-			(effects
-				(font
-					(size 1.27 1.27)
-				)
-			)
-		)
-		(property "Footprint" ""
-			(at 151.13 45.085 0)
-			(effects
-				(font
-					(size 1.27 1.27)
-				)
-				(hide yes)
-			)
-		)
-		(property "Datasheet" "~"
-			(at 151.13 45.085 0)
-			(effects
-				(font
-					(size 1.27 1.27)
-				)
-				(hide yes)
-			)
-		)
-		(property "Description" "Generic connector, double row, 02x06, counter clockwise pin numbering scheme (similar to DIP package numbering), script generated (kicad-library-utils/schlib/autogen/connector/)"
-			(at 151.13 45.085 0)
-			(effects
-				(font
-					(size 1.27 1.27)
-				)
-				(hide yes)
-			)
-		)
-		(pin "8"
-		)
-		(pin "9"
-		)
-		(pin "10"
-		)
-		(pin "7"
-		)
-		(pin "1"
-		)
-		(pin "2"
-		)
-		(pin "3"
-		)
-		(pin "4"
-		)
-		(pin "5"
-		)
-		(pin "6"
-		)
-		(pin "12"
-		)
-		(pin "11"
-		)
-		(instances
-			(project ""
-				(path "/75f9f2a9-074b-4f58-a7a7-2a17dd71988c"
-					(reference "J1")
-					(unit 1)
-				)
-			)
-		)
-	)
-	(symbol
 		(lib_id "power:+3V3")
 		(at 46.355 26.67 0)
@@
 			)
 		)
-		(property "Footprint" "ajm-acorn:Conn_uSDcard"
+		(property "Footprint" "ajm-sdcard:Conn_uSDcard"
 			(at 59.69 140.335 0)
 			(effects
