File: pcbs/diagcard/cptrep-diag-card/cptrep-diag-card.kicad_pcb (KiCad board)
At the start: 2 copper layers, 99.8 x 142.4 mm, 90 parts, among them J2 cpt-backplane_100, J3 Conn_02x04_Counter_Clockwise, J4 Conn_02x04_Counter_Clockwise, J5 Conn_02x04_Counter_Clockwise, J6 Conn_02x04_Counter_Clockwise, J7 Conn_02x04_Counter_Clockwise, J8 Conn_01x08_Pin, J9 Conn_02x24_Counter_Clockwise

Commit message: "Update"
Parts:
- added J10: Conn_02x06_Odd_Even, Connector_PinHeader_2.54mm:PinHeader_2x06_P2.54mm_Vertical, F.Cu at (226.3, 36.3)
- added XS1: 502p_SD_ebay-uSD-push_push_SMD, ajm-sdcard:Conn_uSDcard, F.Cu at (149.5, 67.4)
- moved D1 6.95 mm to (152.9, 56.3), turned to 0 degrees
- moved D2 0.90 mm to (150.2, 81.3)
- moved R56 0.90 mm to (161.3, 81.3)
- moved TR1 0.90 mm to (155.9, 81.3)
Connections:
- J2 pad 1: unconnected-(J2-GND-Pad1) -> GND
- J2 pad 2: unconnected-(J2-GND-Pad2) -> GND
- J2 pad 3: unconnected-(J2-GND-Pad3) -> GND
- J2 pad 4: unconnected-(J2-GND-Pad4) -> GND
Routing:
- net GND: track 377.3 -> 619.7 mm, vias 23 -> 27
- net SD_DAT2: track 0.00 -> 153.9 mm, vias 0 -> 10
- net MISO_DO: track 0.00 -> 128.7 mm, vias 0 -> 6
- net SD_DAT1: track 0.00 -> 124.1 mm, vias 0 -> 4
- net SD_SS: track 0.00 -> 123.7 mm, vias 0 -> 6
- net SD_CLK: track 0.00 -> 122.3 mm, vias 0 -> 4
- net MOSI_DI: track 0.00 -> 121.4 mm, vias 0 -> 6
- net /GPIO16: track 0.00 -> 88.2 mm, vias 0 -> 4
- net /GPIO21: track 0.00 -> 85.6 mm, vias 0 -> 1
- net /GPIO18: track 0.00 -> 85.1 mm, vias 0 -> 4
- net /GPIO19: track 0.00 -> 80.9 mm, vias 0 -> 5
- net /GPIO20: track 0.00 -> 80.1 mm, vias 0 -> 1
- net /GPIO22: track 0.00 -> 78.9 mm, vias 0 -> 3
- net +3.3V: track 85.6 -> 111.5 mm, vias 3 -> 4
- net +5V: track 195.9 -> 217.3 mm
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Other:
- outline, holes or cut-outs redrawn
- board text added: "BOUT BIN TC EOF GP26 GP17 GP15 GP14"
- board text added: "DREQ0 DREQ1 DACK0 DACK1 GP26 GP17 GP15 GP14"
- board text added: "DREQ2 DREQ3 DACK2 DACK3 GP26 GP17 GP15 GP14"
- board text added: "GPIO0"
- board text added: "GPIO1"
- board text added: "GPIO10"
- board text added: "GPIO11"
- board text added: "GPIO20"
- board text added: "GPIO21"
- board text added: "GPIO30"
- board text added: "GPIO31"
- board text added: "GPIO40"
- board text added: "GPIO41"
- board text added: "GPIO47"
- board text added: "HLDACK RESET READY WAIT GP26 GP17 GP15 GP14"
- board text added: "LED0"
- board text added: "LED1"
- board text added: "LED2"
- board text added: "LED3"
- board text added: "LED4"
- board text added: "LED5"
- board text added: "LED6"
- board text added: "LED7"
- board text added: "REF GP26 GP17 GP15 GP14"

Commit message: "Update"
Other:
- board text added: "CPT 8500 Diagnostic Card V1.0 March 2026 menadue@gmail.com"
- board text added: "Jumper for SD card Ensure GP22,GP21,GP20, GP19,GP18,GP16 are free"
Changed lines of the file:
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@@
+		)
+	)
+	(gr_text "Jumper for SD card\nEnsure GP22,GP21,GP20,\nGP19,GP18,GP16 are free"
+		(at 218.44 40.894 90)
+		(layer "F.SilkS")
+		(effects
+			(font
+				(size 1 1)
+				(thickness 0.1)
+			)
+			(justify left bottom)
 		)
 	)
@@
 		(layer "F.SilkS")
 		(effects
+			(font
+				(size 1 1)
+				(thickness 0.1)
+			)
+			(justify left bottom)
+		)
+	)
+	(gr_text "CPT 8500 Diagnostic Card\nV1.0 March 2026\nmenadue@gmail.com"
+		(at 195.464 83.439 0)
+		(layer "F.SilkS")
+		(effects
